Commit message: Turn IMU 180 degrees around the base yaw axis

File: urdf/upkie.urdf (robot description, URDF)
Before this commit: robot upkie, 39 links, 38 joints
Joints:
- joint imu_fix: origin xyz=0 0 0 rpy=0 0 0 -> xyz=0 0 0 rpy=0 0 3.141592653589793

Commit message: Rename chassis to torso

File: urdf/upkie.urdf (robot description, URDF)
Before this commit: robot upkie, 39 links, 38 joints
Links:
- removed link chassis
- added link torso, mass 1.0; collision box size=0.125 0.17 0.25; visual box size=0.125 0.17 0.25
Joints:
- removed joint chassis_fix
- added joint torso_fix: type fixed, parent base, child torso, origin xyz=0 0 -0.1 rpy=0 0 0
- joint battery_fix: parent chassis -> torso
- joint handle_fix: parent chassis -> torso
- joint left_hip_qdd100_stator_fix: parent chassis -> torso
- joint right_hip_qdd100_stator_fix: parent chassis -> torso
