Commit message: Add IMU link

File: urdf/rhea.urdf (robot description, URDF)
Before this commit: robot rhea, 7 links, 6 joints
Links:
- added link imu
Joints:
- added joint imu: type fixed, parent base_link, child imu, origin xyz=0 0 0 rpy=0 0 0

Commit message: Change link names

File: urdf/rhea.urdf (robot description, URDF)
Before this commit: robot rhea, 8 links, 7 joints
Links:
- removed link leg_1_l
- removed link leg_1_r
- removed link leg_2_l
- removed link leg_2_r
- removed link wheel_l
- removed link wheel_r
- added link left_hip, mass 0.1; visual mesh filename=../meshes/dae/simple_bot_mesh.006.dae scale=1.0 1.0 1.0
- added link left_knee, mass 0.1; collision cylinder length=0.02438 radius=0.03428; visual mesh filename=../meshes/dae/simple_bot_mesh.005.dae scale=1.0 1.0 1.0
- added link left_wheel, mass 0.4; collision cylinder length=0.024 radius=0.1; visual mesh filename=../meshes/dae/simple_bot_mesh.004.dae scale=1.0 1.0 1.0
- added link right_hip, mass 0.1; visual mesh filename=../meshes/dae/simple_bot_mesh.003.dae scale=1.0 1.0 1.0
- added link right_knee, mass 0.1; collision cylinder length=0.02438 radius=0.03428; visual mesh filename=../meshes/dae/simple_bot_mesh.002.dae scale=1.0 1.0 1.0
- added link right_wheel, mass 0.4; collision cylinder length=0.024 radius=0.1; visual mesh filename=../meshes/dae/simple_bot_mesh.001.dae scale=1.0 1.0 1.0
Joints:
- removed joint leg_1_l
- removed joint leg_1_r
- removed joint leg_2_l
- removed joint leg_2_r
- removed joint wheel_l
- removed joint wheel_r
- added joint left_hip: type revolute, parent base_link, child left_hip, origin xyz=0 0.1 0 rpy=-1.5708 1.5708 0, axis 0 0 1.0, limit lower=0.5236 upper=1.39626 effort=35.0 velocity=26.0
- added joint left_knee: type revolute, parent left_hip, child left_knee, origin xyz=0.225 0 0 rpy=0 0 0, axis 0 0 1.0, limit lower=-2.79253 upper=-1.0472 effort=35.0 velocity=26.0
- added joint left_wheel: type continuous, parent left_knee, child left_wheel, origin xyz=0.225 0 0 rpy=0 0 0, axis 0 0 1.0, limit effort=9.0 velocity=42.0
- added joint right_hip: type revolute, parent base_link, child right_hip, origin xyz=0 -0.1 0 rpy=1.5708 1.5708 0, axis 0 0 1.0, limit lower=-1.39626 upper=-0.5236 effort=35.0 velocity=26.0
- added joint right_knee: type revolute, parent right_hip, child right_knee, origin xyz=0.225 0 0 rpy=0 0 0, axis 0 0 1.0, limit lower=1.0472 upper=2.79253 effort=35.0 velocity=26.0
- added joint right_wheel: type continuous, parent right_knee, child right_wheel, origin xyz=0.225 0 0 rpy=0 0 0, axis 0 0 1.0, limit effort=9.0 velocity=42.0

Commit message: Correct IMU link inertia and orientation

File: urdf/rhea.urdf (robot description, URDF)
Before this commit: robot rhea, 8 links, 7 joints
Links:
- link imu: mass None -> 0.001
Joints:
- joint imu: origin xyz=0 0 0 rpy=0 0 0 -> xyz=0 0 0 rpy=1.5708 0 1.5708
