Commit message: Update for Rhea v2

File: description/rhea.ros2_control.xacro (robot description, xacro)
@@ -7,5 +7,5 @@
                 <param name="imu_mounting_deg.yaw">90.0</param>
                 <param name="imu_mounting_deg.pitch">0.0</param>
-                <param name="imu_mounting_deg.roll">90.0</param>
+                <param name="imu_mounting_deg.roll">-90.0</param>
             </hardware>
             <joint name="right_hip">
@@ -19,7 +19,33 @@
                 <param name="kd_scale">5.0</param>
                 <param name="axis_direction">-1</param>
-                <param name="position_offset">-1.39626</param>
-                <param name="position_min">-1.39626</param>
-                <param name="position_max">-0.523599</param>
+                <param name="position_offset">-2.46091</param>
+                <param name="position_min">-2.46091</param>
+                <param name="position_max">0.68068</param>
+                <param name="velocity_max">10.0</param>
+                <param name="effort_max">10.0</param>
+                <param name="kp_max">100.0</param>
+                <param name="kd_max">10.0</param>
+                <command_interface name="position"/>
+                <command_interface name="velocity"/>
+                <command_interface name="effort"/>
+                <command_interface name="kp"/>
+                <command_interface name="kd"/>
+                <state_interface name="position"/>
+                <state_interface name="velocity"/>
+                <state_interface name="effort"/>
+            </joint>
+            <joint name="right_knee">
+                <param name="can_channel">1</param>
+                <param name="can_id">2</param>
+                <param name="can_protocol">cheetah</param>
+                <param name="position_scale">95.5</param>
+                <param name="velocity_scale">30.0</param>
+                <param name="effort_scale">18.0</param>
+                <param name="kp_scale">500.0</param>
+                <param name="kd_scale">5.0</param>
+                <param name="axis_direction">-1</param>
+                <param name="position_offset">2.75762</param>
+                <param name="position_min">0.66323</param>
+                <param name="position_max">2.75762</param>
                 <param name="velocity_max">10.0</param>
                 <param name="effort_max">10.0</param>
@@ -37,5 +63,31 @@
             <joint name="right_wheel">
                 <param name="can_channel">1</param>
-                <param name="can_id">2</param>
+                <param name="can_id">3</param>
+                <param name="can_protocol">cheetah</param>
+                <param name="position_scale">12.5</param>
+                <param name="velocity_scale">200.0</param>
+                <param name="effort_scale">18.0</param>
+                <param name="kp_scale">500.0</param>
+                <param name="kd_scale">5.0</param>
+                <param name="axis_direction">-1</param>
+                <param name="position_offset">0.0</param>
+                <param name="position_min">-1.0</param>
+                <param name="position_max">1.0</param>
+                <param name="velocity_max">30.0</param>
+                <param name="effort_max">10.0</param>
+                <param name="kp_max">100.0</param>
+                <param name="kd_max">2.0</param>
+                <command_interface name="position"/>
+                <command_interface name="velocity"/>
+                <command_interface name="effort"/>
+                <command_interface name="kp"/>
+                <command_interface name="kd"/>
+                <state_interface name="position"/>
+                <state_interface name="velocity"/>
+                <state_interface name="effort"/>
+            </joint>
+            <joint name="left_hip">
+                <param name="can_channel">2</param>
+                <param name="can_id">4</param>
                 <param name="can_protocol">cheetah</param>
                 <param name="position_scale">95.5</param>
@@ -45,7 +97,7 @@
                 <param name="kd_scale">5.0</param>
                 <param name="axis_direction">-1</param>
-                <param name="position_offset">0.0</param>
-                <param name="position_min">-1.0</param>
-                <param name="position_max">1.0</param>
+                <param name="position_offset">2.46091</param>
+                <param name="position_min">-0.68068</param>
+                <param name="position_max">2.46091</param>
                 <param name="velocity_max">10.0</param>
                 <param name="effort_max">10.0</param>
@@ -61,7 +113,7 @@
                 <state_interface name="effort"/>
             </joint>
-            <joint name="left_hip">
+            <joint name="left_knee">
                 <param name="can_channel">2</param>
-                <param name="can_id">3</param>
+                <param name="can_id">5</param>
                 <param name="can_protocol">cheetah</param>
                 <param name="position_scale">95.5</param>
@@ -71,7 +123,7 @@
                 <param name="kd_scale">5.0</param>
                 <param name="axis_direction">-1</param>
-                <param name="position_offset">1.39626</param>
-                <param name="position_min">0.523599</param>
-                <param name="position_max">1.39626</param>
+                <param name="position_offset">-2.75762</param>
+                <param name="position_min">-2.75762</param>
+                <param name="position_max">-0.66323</param>
                 <param name="velocity_max">10.0</param>
                 <param name="effort_max">10.0</param>
@@ -89,8 +141,8 @@
             <joint name="left_wheel">
                 <param name="can_channel">2</param>
-                <param name="can_id">4</param>
+                <param name="can_id">6</param>
                 <param name="can_protocol">cheetah</param>
-                <param name="position_scale">95.5</param>
-                <param name="velocity_scale">30.0</param>
+                <param name="position_scale">12.5</param>
+                <param name="velocity_scale">200.0</param>
                 <param name="effort_scale">18.0</param>
                 <param name="kp_scale">500.0</param>
@@ -100,6 +152,6 @@
                 <param name="position_min">-1.0</param>
                 <param name="position_max">1.0</param>
-                <param name="velocity_max">10.0</param>
-                <param name="effort_max">10.0</param>
+                <param name="velocity_max">30.0</param>
+                <param name="effort_max">2.0</param>
                 <param name="kp_max">100.0</param>
                 <param name="kd_max">10.0</param>

File: description/urdf/rhea.urdf (robot description, URDF)
Before this commit: robot rhea, 8 links, 7 joints
Links:
- link base_link: mass 3.0 -> 4.0; geometry collision box size=0.216 0.14 0.231; visual mesh filename=package://rhea_description/meshes/dae/rheav2.dae scale=1.0 1.0 1.0
- link left_hip: mass 0.1 -> 1.0; geometry collision box size=0.05693 0.0756 0.30004; visual mesh filename=package://rhea_description/meshes/dae/rheav2.006.dae scale=1.0 1.0 1.0
- link left_knee: mass 0.1 -> 0.5; geometry collision box size=0.05693 0.028 0.30004; visual mesh filename=package://rhea_description/meshes/dae/rheav2.004.dae scale=1.0 1.0 1.0
- link left_wheel: mass 0.4 -> 1.0; geometry collision cylinder length=0.048 radius=0.11; visual mesh filename=package://rhea_description/meshes/dae/rheav2.005.dae scale=1.0 1.0 1.0
- link right_hip: mass 0.1 -> 1.0; geometry collision box size=0.05693 0.0756 0.30004; visual mesh filename=package://rhea_description/meshes/dae/rheav2.003.dae scale=1.0 1.0 1.0
- link right_knee: mass 0.1 -> 0.5; geometry collision box size=0.05693 0.028 0.30004; visual mesh filename=package://rhea_description/meshes/dae/rheav2.001.dae scale=1.0 1.0 1.0
- link right_wheel: mass 0.4 -> 1.0; geometry collision cylinder length=0.048 radius=0.11; visual mesh filename=package://rhea_description/meshes/dae/rheav2.002.dae scale=1.0 1.0 1.0
Joints:
- joint imu: origin xyz=0 0 0 rpy=1.5708 0 1.5708 -> xyz=0 0 0 rpy=1.5708 0 -1.5708
- joint left_hip: limit lower=0.5236 upper=1.39626 effort=35.0 velocity=26.0 -> lower=-0.68068 upper=2.46091 effort=35.0 velocity=26.0; origin xyz=0 0.1 0 rpy=-1.5708 1.5708 0 -> xyz=0 0.1255 0 rpy=-1.5708 1.5708 0
- joint left_knee: limit lower=-2.79253 upper=-1.0472 effort=35.0 velocity=26.0 -> lower=-2.75762 upper=-0.66323 effort=35.0 velocity=26.0; origin xyz=0.225 0 0 rpy=0 0 0 -> xyz=0.25 0 0 rpy=0 0 0
- joint left_wheel: limit effort=9.0 velocity=42.0 -> effort=2.0 velocity=250.0; origin xyz=0.225 0 0 rpy=0 0 0 -> xyz=0.25 0 0 rpy=0 0 0
- joint right_hip: limit lower=-1.39626 upper=-0.5236 effort=35.0 velocity=26.0 -> lower=-2.46091 upper=0.68068 effort=35.0 velocity=26.0; origin xyz=0 -0.1 0 rpy=1.5708 1.5708 0 -> xyz=0 -0.1255 0 rpy=1.5708 1.5708 0
- joint right_knee: limit lower=1.0472 upper=2.79253 effort=35.0 velocity=26.0 -> lower=0.66323 upper=2.75762 effort=35.0 velocity=26.0; origin xyz=0.225 0 0 rpy=0 0 0 -> xyz=0.25 0 0 rpy=0 0 0
- joint right_wheel: limit effort=9.0 velocity=42.0 -> effort=2.0 velocity=250.0; origin xyz=0.225 0 0 rpy=0 0 0 -> xyz=0.25 0 0 rpy=0 0 0
